File: Board/Ackbar.kicad_sch (KiCad schematic)
At the start: 9 parts, among them J1 TOF, J2 GNSS, J3 HALL, J4 MOTOR, J5 PWR_IN, J6 EPD, U1 ESP32-S3 Pico, U2 VREG, U3 TMC2209

Commit message: Cleanup
Parts:
- U1: footprint Akbar:Waveshare ESP32-S3 Pico -> Ackbar:Waveshare ESP32-S3 Pico; symbol Akbar:Waveshare_ESP32-S3_Pico -> Ackbar:Waveshare_ESP32-S3_Pico
- U2: footprint Akbar:Buck Regulator -> Ackbar:Buck Regulator; symbol Akbar:Buck_Regulator -> Ackbar:Buck_Regulator
- U3: footprint Akbar:BTT TMC2209 -> Ackbar:BTT TMC2209; symbol Akbar:BTT_TMC2209 -> Ackbar:BTT_TMC2209
Changed lines of the file:
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@@
     (pin "2")
     (instances
-      (project "Akbar"
+      (project "Ackbar"
         (path "/10d22af5-0d05-45a6-b4a8-43aad0d497f4"
           (reference "J5") (unit 1)
@@
     (pin "5")
     (instances
-      (project "Akbar"
+      (project "Ackbar"
         (path "/10d22af5-0d05-45a6-b4a8-43aad0d497f4"
           (reference "J2") (unit 1)
@@
     )
   )
-  (symbol (lib_id "Akbar:Waveshare_ESP32-S3_Pico") (at 111.76 38.1 0) (unit 1)
+  (symbol (lib_id "Ackbar:Waveshare_ESP32-S3_Pico") (at 111.76 38.1 0) (unit 1)
     (in_bom yes) (on_board yes) (dnp no)
     (property "Reference" "U1" (at 111.76 30.48 0)
@@
       (effects (font (size 1.27 1.27)))
     )
-    (property "Footprint" "Akbar:Waveshare ESP32-S3 Pico" (at 111.76 38.1 0)
+    (property "Footprint" "Ackbar:Waveshare ESP32-S3 Pico" (at 111.76 38.1 0)
       (effects (font (size 1.27 1.27)) hide)
     )
@@
     (pin "9")
     (instances
-      (project "Akbar"
+      (project "Ackbar"
         (path "/10d22af5-0d05-45a6-b4a8-43aad0d497f4"
           (reference "U1") (unit 1)
@@
     )
   )
-  (symbol (lib_id "Akbar:Buck_Regulator") (at 111.76 153.67 180) (unit 1)
+  (symbol (lib_id "Ackbar:Buck_Regulator") (at 111.76 153.67 180) (unit 1)
     (in_bom yes) (on_board yes) (dnp no) (fields_autoplaced)
     (property "Reference" "U2" (at 100.33 153.035 0)
@@
       (effects (font (size 1.27 1.27)))
     )
-    (property "Footprint" "Akbar:Buck Regulator" (at 111.76 153.67 0)
+    (property "Footprint" "Ackbar:Buck Regulator" (at 111.76 153.67 0)
       (effects (font (size 1.27 1.27)) hide)
     )
@@
     (pin "4")
     (instances
-      (project "Akbar"
+      (project "Ackbar"
         (path "/10d22af5-0d05-45a6-b4a8-43aad0d497f4"
           (reference "U2") (unit 1)
@@
     )
   )
-  (symbol (lib_id "Akbar:BTT_TMC2209") (at 111.76 109.22 0) (unit 1)
+  (symbol (lib_id "Ackbar:BTT_TMC2209") (at 111.76 109.22 0) (unit 1)
     (in_bom yes) (on_board yes) (dnp no)
     (property "Reference" "U3" (at 111.76 138.43 0)
@@
       (effects (font (size 1.27 1.27)))
     )
-    (property "Footprint" "Akbar:BTT TMC2209" (at 111.76 109.22 0)
+    (property "Footprint" "Ackbar:BTT TMC2209" (at 111.76 109.22 0)
       (effects (font (size 1.27 1.27)) hide)
     )
@@
     (pin "9")
     (instances
-      (project "Akbar"
+      (project "Ackbar"
         (path "/10d22af5-0d05-45a6-b4a8-43aad0d497f4"
           (reference "U3") (unit 1)
@@
     (pin "5")
     (instances
-      (project "Akbar"
+      (project "Ackbar"
         (path "/10d22af5-0d05-45a6-b4a8-43aad0d497f4"
           (reference "J1") (unit 1)
@@
     (pin "3")
     (instances
-      (project "Akbar"
+      (project "Ackbar"
         (path "/10d22af5-0d05-45a6-b4a8-43aad0d497f4"
           (reference "J3") (unit 1)
@@
     (pin "4")
     (instances
-      (project "Akbar"
+      (project "Ackbar"
         (path "/10d22af5-0d05-45a6-b4a8-43aad0d497f4"
           (reference "J4") (unit 1)
@@
     (pin "8")
     (instances
-      (project "Akbar"
+      (project "Ackbar"
         (path "/10d22af5-0d05-45a6-b4a8-43aad0d497f4"
           (reference "J6") (unit 1)

Commit message: add inverter to schematic
Parts:
- added U4: SN74LVC1G04DCKR, Ackbar:SOT65P210X110-5N, symbol Ackbar:SN74LVC1G04DCKR
Connections:
- net GND: now also U4.3 (GND)
- net VBUS: no longer names the net of U1.40 (VBUS)
- net VBUS: now also U4.2 (A), U4.5 (VCC); no longer U2.4 (EN)
- new net: U2.4 (EN), U4.4 (Y)
Changed lines of the file:
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@@
 (kicad_sch (version 20230121) (generator eeschema)
   (paper "A4")
+  (junction (at 138.43 149.86) (diameter 0) (color 0 0 0 0)
+  )
+  (junction (at 193.04 153.67) (diameter 0) (color 0 0 0 0)
+  )
   (wire (pts (xy 134.62 147.32) (xy 123.19 147.32))
     (stroke (width 0) (type default))
@@
     (stroke (width 0) (type default))
   )
+  (wire (pts (xy 153.67 144.78) (xy 138.43 144.78))
+    (stroke (width 0) (type default))
+  )
   (wire (pts (xy 123.19 68.58) (xy 160.02 68.58))
     (stroke (width 0) (type default))
@@
     (stroke (width 0) (type default))
   )
+  (wire (pts (xy 153.67 148.59) (xy 153.67 144.78))
+    (stroke (width 0) (type default))
+  )
   (wire (pts (xy 99.06 128.27) (xy 92.71 128.27))
     (stroke (width 0) (type default))
@@
     (stroke (width 0) (type default))
   )
+  (wire (pts (xy 193.04 163.83) (xy 193.04 153.67))
+    (stroke (width 0) (type default))
+  )
   (wire (pts (xy 90.17 71.12) (xy 100.33 71.12))
     (stroke (width 0) (type default))
   )
+  (wire (pts (xy 138.43 144.78) (xy 138.43 149.86))
+    (stroke (width 0) (type default))
+  )
   (wire (pts (xy 59.69 48.26) (xy 71.12 48.26))
     (stroke (width 0) (type default))
@@
     (stroke (width 0) (type default))
   )
+  (wire (pts (xy 123.19 40.64) (xy 193.04 40.64))
+    (stroke (width 0) (type default))
+  )
   (wire (pts (xy 123.19 45.72) (xy 129.54 45.72))
     (stroke (width 0) (type default))
   )
+  (wire (pts (xy 99.06 120.65) (xy 92.71 120.65))
+    (stroke (width 0) (type default))
+  )
+  (wire (pts (xy 90.17 73.66) (xy 100.33 73.66))
+    (stroke (width 0) (type default))
+  )
+  (wire (pts (xy 130.81 130.81) (xy 124.46 130.81))
+    (stroke (width 0) (type default))
+  )
+  (wire (pts (xy 90.17 66.04) (xy 100.33 66.04))
+    (stroke (width 0) (type default))
+  )
+  (wire (pts (xy 140.97 53.34) (xy 160.02 53.34))
+    (stroke (width 0) (type default))
+  )
+  (wire (pts (xy 59.69 53.34) (xy 71.12 53.34))
+    (stroke (width 0) (type default))
+  )
+  (wire (pts (xy 59.69 43.18) (xy 71.12 43.18))
+    (stroke (width 0) (type default))
+  )
+  (wire (pts (xy 123.19 53.34) (xy 129.54 53.34))
+    (stroke (width 0) (type default))
+  )
+  (wire (pts (xy 130.81 115.57) (xy 124.46 115.57))
+    (stroke (width 0) (type default))
+  )
+  (wire (pts (xy 107.95 100.33) (xy 107.95 104.14))
+    (stroke (width 0) (type default))
+  )
+  (wire (pts (xy 148.59 66.04) (xy 160.02 66.04))
+    (stroke (width 0) (type default))
+  )
+  (wire (pts (xy 148.59 76.2) (xy 160.02 76.2))
+    (stroke (width 0) (type default))
+  )
+  (wire (pts (xy 124.46 120.65) (xy 138.43 120.65))
+    (stroke (width 0) (type default))
+  )
+  (wire (pts (xy 90.17 58.42) (xy 100.33 58.42))
+    (stroke (width 0) (type default))
+  )
+  (wire (pts (xy 90.17 68.58) (xy 100.33 68.58))
+    (stroke (width 0) (type default))
+  )
+  (wire (pts (xy 130.81 118.11) (xy 124.46 118.11))
+    (stroke (width 0) (type default))
+  )
   (wire (pts (xy 123.19 149.86) (xy 138.43 149.86))
     (stroke (width 0) (type default))
   )
-  (wire (pts (xy 99.06 120.65) (xy 92.71 120.65))
-    (stroke (width 0) (type default))
-  )
-  (wire (pts (xy 90.17 73.66) (xy 100.33 73.66))
-    (stroke (width 0) (type default))
-  )
-  (wire (pts (xy 130.81 130.81) (xy 124.46 130.81))
-    (stroke (width 0) (type default))
-  )
-  (wire (pts (xy 123.19 40.64) (xy 129.54 40.64))
-    (stroke (width 0) (type default))
-  )
-  (wire (pts (xy 90.17 66.04) (xy 100.33 66.04))
-    (stroke (width 0) (type default))
-  )
-  (wire (pts (xy 140.97 53.34) (xy 160.02 53.34))
-    (stroke (width 0) (type default))
-  )
-  (wire (pts (xy 59.69 53.34) (xy 71.12 53.34))
-    (stroke (width 0) (type default))
-  )
-  (wire (pts (xy 59.69 43.18) (xy 71.12 43.18))
-    (stroke (width 0) (type default))
-  )
-  (wire (pts (xy 123.19 53.34) (xy 129.54 53.34))
-    (stroke (width 0) (type default))
-  )
-  (wire (pts (xy 130.81 115.57) (xy 124.46 115.57))
-    (stroke (width 0) (type default))
-  )
-  (wire (pts (xy 107.95 100.33) (xy 107.95 104.14))
-    (stroke (width 0) (type default))
-  )
-  (wire (pts (xy 148.59 66.04) (xy 160.02 66.04))
-    (stroke (width 0) (type default))
-  )
-  (wire (pts (xy 148.59 76.2) (xy 160.02 76.2))
-    (stroke (width 0) (type default))
-  )
-  (wire (pts (xy 124.46 120.65) (xy 138.43 120.65))
-    (stroke (width 0) (type default))
-  )
-  (wire (pts (xy 90.17 58.42) (xy 100.33 58.42))
-    (stroke (width 0) (type default))
-  )
-  (wire (pts (xy 90.17 68.58) (xy 100.33 68.58))
-    (stroke (width 0) (type default))
-  )
-  (wire (pts (xy 130.81 118.11) (xy 124.46 118.11))
-    (stroke (width 0) (type default))
-  )
   (wire (pts (xy 123.19 55.88) (xy 129.54 55.88))
     (stroke (width 0) (type default))
   )
+  (wire (pts (xy 193.04 40.64) (xy 193.04 153.67))
+    (stroke (width 0) (type default))
+  )
   (wire (pts (xy 107.95 100.33) (xy 92.71 100.33))
     (stroke (width 0) (type default))
@@
     (stroke (width 0) (type default))
   )
+  (wire (pts (xy 157.48 163.83) (xy 193.04 163.83))
+    (stroke (width 0) (type default))
+  )
+  (wire (pts (xy 157.48 154.94) (xy 157.48 153.67))
+    (stroke (width 0) (type default))
+  )
   (wire (pts (xy 90.17 60.96) (xy 100.33 60.96))
     (stroke (width 0) (type default))
@@
     (stroke (width 0) (type default))
   )
+  (wire (pts (xy 123.19 154.94) (xy 157.48 154.94))
+    (stroke (width 0) (type default))
+  )
   (wire (pts (xy 123.19 86.36) (xy 140.97 86.36))
     (stroke (width 0) (type default))
@@
     (stroke (width 0) (type default))
   )
-  (wire (pts (xy 123.19 154.94) (xy 134.62 154.94))
-    (stroke (width 0) (type default))
-  )
   (wire (pts (xy 148.59 60.96) (xy 160.02 60.96))
     (stroke (width 0) (type default))
@@
     (stroke (width 0) (type default))
   )
+  (wire (pts (xy 157.48 148.59) (xy 153.67 148.59))
+    (stroke (width 0) (type default))
+  )
   (wire (pts (xy 124.46 125.73) (xy 138.43 125.73))
     (stroke (width 0) (type default))
@@
     (stroke (width 0) (type default))
   )
+  (wire (pts (xy 157.48 158.75) (xy 157.48 163.83))
+    (stroke (width 0) (type default))
+  )
   (label "M_B1" (at 127 125.73 0) (fields_autoplaced)
     (effects (font (size 1.27 1.27)) (justify left bottom))
@@
     (effects (font (size 1.27 1.27)) (justify left bottom))
   )
-  (label "VBUS" (at 125.73 40.64 0) (fields_autoplaced)
-    (effects (font (size 1.27 1.27)) (justify left bottom))
-  )
   (label "STP_MS3" (at 99.06 123.19 180) (fields_autoplaced)
     (effects (font (size 1.27 1.27)) (justify right bottom))
@@
   (label "M_A1" (at 127 123.19 0) (fields_autoplaced)
     (effects (font (size 1.27 1.27)) (justify left bottom))
-  )
-  (label "VBUS" (at 134.62 154.94 180) (fields_autoplaced)
-    (effects (font (size 1.27 1.27)) (justify right bottom))
   )
   (label "SCL" (at 148.59 48.26 0) (fields_autoplaced)
@@
         )
       )
+    )
+  )
+  (symbol (lib_id "Ackbar:SN74LVC1G04DCKR") (at 175.26 153.67 180) (unit 1)
+    (in_bom yes) (on_board yes) (dnp no) (fields_autoplaced)
+    (property "Reference" "U4" (at 175.26 140.97 0)
+      (effects (font (size 1.27 1.27)))
+    )
+    (property "Value" "SN74LVC1G04DCKR" (at 175.26 143.51 0)
+      (effects (font (size 1.27 1.27)))
+    )
+    (property "Footprint" "Ackbar:SOT65P210X110-5N" (at 175.26 153.67 0)
+      (effects (font (size 1.27 1.27)) (justify bottom) hide)
+    )
+    (property "Datasheet" "" (at 175.26 153.67 0)
+      (effects (font (size 1.27 1.27)) hide)
+    )
+    (property "DigiKey_Part_Number" "296-11600-2-ND" (at 175.26 153.67 0)
+      (effects (font (size 1.27 1.27)) (justify bottom) hide)
+    )
+    (property "MF" "Texas Instruments" (at 175.26 153.67 0)
+      (effects (font (size 1.27 1.27)) (justify bottom) hide)
+    )
+    (property "Purchase-URL" "https://www.snapeda.com/api/url_track_click_mouser/?unipart_id=359755&manufacturer=Texas Instruments&part_name=SN74LVC1G04DCKR&search_term=None" (at 175.26 153.67 0)
+      (effects (font (size 1.27 1.27)) (justify bottom) hide)
+    )
+    (property "Package" "SC70-5 Texas Instruments" (at 175.26 153.67 0)
+      (effects (font (size 1.27 1.27)) (justify bottom) hide)
+    )
+    (property "SnapEDA_Link" "https://www.snapeda.com/parts/SN74LVC1G04DCKR/Texas+Instruments/view-part/?ref=snap" (at 175.26 153.67 0)
+      (effects (font (size 1.27 1.27)) (justify bottom) hide)
+    )
+    (property "MP" "SN74LVC1G04DCKR" (at 175.26 153.67 0)
+      (effects (font (size 1.27 1.27)) (justify bottom) hide)
+    )
+    (property "Description" "\nSingle 1.65-V to 5.5-V inverter\n" (at 175.26 153.67 0)
+      (effects (font (size 1.27 1.27)) (justify bottom) hide)
+    )
+    (property "Check_prices" "https://www.snapeda.com/parts/SN74LVC1G04DCKR/Texas+Instruments/view-part/?ref=eda" (at 175.26 153.67 0)
+      (effects (font (size 1.27 1.27)) (justify bottom) hide)
+    )
+    (pin "2")
+    (pin "3")
+    (pin "4")
+    (pin "5")
+    (instances
+      (project "Ackbar"
+        (path "/10d22af5-0d05-45a6-b4a8-43aad0d497f4"
+          (reference "U4") (unit 1)
+        )
+      )

Commit message: Larger footprint for inverter
Parts:
- U4: value SN74LVC1G04DCKR -> SN74LVC1G04; footprint Ackbar:SOT65P210X110-5N -> Ackbar:SOT95P280X145-5N
Changed lines of the file:
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@@
       (effects (font (size 1.27 1.27)))
     )
-    (property "Value" "SN74LVC1G04DCKR" (at 175.26 143.51 0)
+    (property "Value" "SN74LVC1G04" (at 175.26 143.51 0)
       (effects (font (size 1.27 1.27)))
     )
-    (property "Footprint" "Ackbar:SOT65P210X110-5N" (at 175.26 153.67 0)
+    (property "Footprint" "Ackbar:SOT95P280X145-5N" (at 175.26 153.67 0)
       (effects (font (size 1.27 1.27)) (justify bottom) hide)
     )

Commit message: cleanup vreg inhibit
Connections:
- net at U1.37 (3V3_EN): now also U4.2 (A)
- net at U1.39 (VSYS): now also U4.5 (VCC)
- now unconnected: U1.40 (VBUS)
Changed lines of the file:
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@@
   (junction (at 138.43 149.86) (diameter 0) (color 0 0 0 0)
   )
-  (junction (at 193.04 153.67) (diameter 0) (color 0 0 0 0)
-  )
   (wire (pts (xy 134.62 147.32) (xy 123.19 147.32))
     (stroke (width 0) (type default))
@@
     (stroke (width 0) (type default))
   )
+  (wire (pts (xy 135.89 43.18) (xy 135.89 35.56))
+    (stroke (width 0) (type default))
+  )
   (wire (pts (xy 90.17 53.34) (xy 100.33 53.34))
     (stroke (width 0) (type default))
@@
     (stroke (width 0) (type default))
   )
-  (wire (pts (xy 193.04 163.83) (xy 193.04 153.67))
-    (stroke (width 0) (type default))
-  )
   (wire (pts (xy 90.17 71.12) (xy 100.33 71.12))
     (stroke (width 0) (type default))
@@
     (stroke (width 0) (type default))
   )
+  (wire (pts (xy 193.04 153.67) (xy 193.04 39.37))
+    (stroke (width 0) (type default))
+  )
   (wire (pts (xy 59.69 48.26) (xy 71.12 48.26))
     (stroke (width 0) (type default))
@@
     (stroke (width 0) (type default))
   )
-  (wire (pts (xy 123.19 40.64) (xy 193.04 40.64))
+  (wire (pts (xy 135.89 35.56) (xy 196.85 35.56))
     (stroke (width 0) (type default))
   )
@@
     (stroke (width 0) (type default))
   )
+  (wire (pts (xy 139.7 39.37) (xy 139.7 48.26))
+    (stroke (width 0) (type default))
+  )
+  (wire (pts (xy 196.85 35.56) (xy 196.85 163.83))
+    (stroke (width 0) (type default))
+  )
   (wire (pts (xy 99.06 120.65) (xy 92.71 120.65))
     (stroke (width 0) (type default))
@@
     (stroke (width 0) (type default))
   )
-  (wire (pts (xy 193.04 40.64) (xy 193.04 153.67))
-    (stroke (width 0) (type default))
-  )
   (wire (pts (xy 107.95 100.33) (xy 92.71 100.33))
     (stroke (width 0) (type default))
@@
     (stroke (width 0) (type default))
   )
+  (wire (pts (xy 139.7 48.26) (xy 123.19 48.26))
+    (stroke (width 0) (type default))
+  )
   (wire (pts (xy 148.59 45.72) (xy 160.02 45.72))
     (stroke (width 0) (type default))
@@
     (stroke (width 0) (type default))
   )
-  (wire (pts (xy 157.48 163.83) (xy 193.04 163.83))
-    (stroke (width 0) (type default))
-  )
   (wire (pts (xy 157.48 154.94) (xy 157.48 153.67))
     (stroke (width 0) (type default))
@@
     (stroke (width 0) (type default))
   )
+  (wire (pts (xy 152.4 163.83) (xy 152.4 158.75))
+    (stroke (width 0) (type default))
+  )
   (wire (pts (xy 148.59 50.8) (xy 160.02 50.8))
     (stroke (width 0) (type default))
@@
     (stroke (width 0) (type default))
   )
+  (wire (pts (xy 193.04 39.37) (xy 139.7 39.37))
+    (stroke (width 0) (type default))
+  )
+  (wire (pts (xy 152.4 158.75) (xy 157.48 158.75))
+    (stroke (width 0) (type default))
+  )
   (wire (pts (xy 148.59 60.96) (xy 160.02 60.96))
     (stroke (width 0) (type default))
@@
     (stroke (width 0) (type default))
   )
+  (wire (pts (xy 196.85 163.83) (xy 152.4 163.83))
+    (stroke (width 0) (type default))
+  )
+  (wire (pts (xy 123.19 43.18) (xy 135.89 43.18))
+    (stroke (width 0) (type default))
+  )
   (wire (pts (xy 59.69 40.64) (xy 71.12 40.64))
     (stroke (width 0) (type default))
   )
-  (wire (pts (xy 157.48 158.75) (xy 157.48 163.83))
-    (stroke (width 0) (type default))
-  )

Commit message: WIP of firmware refactoring
Parts:
- added R1: 1K, Resistor_SMD:R_0805_2012Metric_Pad1.20x1.40mm_HandSolder, symbol Device:R_US
Connections:
- net STP_MS3: now also R1.1
- net STP_PDN: now also R1.2
Changed lines of the file:
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@@
     (stroke (width 0) (type default))
   )
-  (wire (pts (xy 99.06 125.73) (xy 92.71 125.73))
+  (wire (pts (xy 86.36 125.73) (xy 99.06 125.73))
     (stroke (width 0) (type default))
   )
@@
     (stroke (width 0) (type default))
   )
+  (wire (pts (xy 86.36 123.19) (xy 86.36 120.65))
+    (stroke (width 0) (type default))
+  )
   (wire (pts (xy 193.04 153.67) (xy 193.04 39.37))
     (stroke (width 0) (type default))
@@
     (stroke (width 0) (type default))
   )
+  (wire (pts (xy 86.36 120.65) (xy 78.74 120.65))
+    (stroke (width 0) (type default))
+  )
   (wire (pts (xy 59.69 43.18) (xy 71.12 43.18))
     (stroke (width 0) (type default))
@@
     (stroke (width 0) (type default))
   )
-  (wire (pts (xy 99.06 123.19) (xy 92.71 123.19))
+  (wire (pts (xy 86.36 123.19) (xy 99.06 123.19))
     (stroke (width 0) (type default))
   )
@@
     (stroke (width 0) (type default))
   )
+  (wire (pts (xy 86.36 128.27) (xy 78.74 128.27))
+    (stroke (width 0) (type default))
+  )
   (wire (pts (xy 148.59 60.96) (xy 160.02 60.96))
     (stroke (width 0) (type default))
@@
   )
   (wire (pts (xy 124.46 125.73) (xy 138.43 125.73))
+    (stroke (width 0) (type default))
+  )
+  (wire (pts (xy 86.36 125.73) (xy 86.36 128.27))
     (stroke (width 0) (type default))
   )
@@
         )
       )
+    )
+  )
+  (symbol (lib_id "Device:R_US") (at 78.74 124.46 0) (unit 1)
+    (in_bom yes) (on_board yes) (dnp no) (fields_autoplaced)
+    (property "Reference" "R1" (at 81.28 123.19 0)
+      (effects (font (size 1.27 1.27)) (justify left))
+    )
+    (property "Value" "1K" (at 81.28 125.73 0)
+      (effects (font (size 1.27 1.27)) (justify left))
+    )
+    (property "Footprint" "Resistor_SMD:R_0805_2012Metric_Pad1.20x1.40mm_HandSolder" (at 79.756 124.714 90)
+      (effects (font (size 1.27 1.27)) hide)
+    )
+    (property "Datasheet" "~" (at 78.74 124.46 0)
+      (effects (font (size 1.27 1.27)) hide)
+    )
+    (pin "1")
+    (pin "2")
+    (instances
+      (project "Ackbar"
+        (path "/10d22af5-0d05-45a6-b4a8-43aad0d497f4"
+          (reference "R1") (unit 1)
+        )
+      )

Commit message: Add pullup resistor to vreg enable
Parts:
- added R2: 1K, Resistor_SMD:R_0805_2012Metric_Pad1.20x1.40mm_HandSolder, symbol Device:R_US
Connections:
- net VIN: now also R2.1
- net at U2.4 (EN), U4.4 (Y): now also R2.2
Changed lines of the file:
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@@
   (junction (at 138.43 149.86) (diameter 0) (color 0 0 0 0)
   )
+  (junction (at 130.81 160.02) (diameter 0) (color 0 0 0 0)
+  )
+  (junction (at 130.81 152.4) (diameter 0) (color 0 0 0 0)
+  )
   (wire (pts (xy 134.62 147.32) (xy 123.19 147.32))
     (stroke (width 0) (type default))
@@
     (stroke (width 0) (type default))
   )
+  (wire (pts (xy 130.81 160.02) (xy 139.7 160.02))
+    (stroke (width 0) (type default))
+  )
   (wire (pts (xy 123.19 71.12) (xy 129.54 71.12))
     (stroke (width 0) (type default))
@@
     (stroke (width 0) (type default))
   )
+  (wire (pts (xy 139.7 160.02) (xy 139.7 154.94))
+    (stroke (width 0) (type default))
+  )
   (wire (pts (xy 123.19 68.58) (xy 160.02 68.58))
     (stroke (width 0) (type default))
@@
     (stroke (width 0) (type default))
   )
+  (wire (pts (xy 123.19 160.02) (xy 130.81 160.02))
+    (stroke (width 0) (type default))
+  )
   (wire (pts (xy 90.17 50.8) (xy 100.33 50.8))
     (stroke (width 0) (type default))
@@
     (stroke (width 0) (type default))
   )
+  (wire (pts (xy 123.19 154.94) (xy 123.19 160.02))
+    (stroke (width 0) (type default))
+  )
   (wire (pts (xy 90.17 73.66) (xy 100.33 73.66))
     (stroke (width 0) (type default))
@@
     (stroke (width 0) (type default))
   )
+  (wire (pts (xy 139.7 154.94) (xy 157.48 154.94))
+    (stroke (width 0) (type default))
+  )
   (wire (pts (xy 148.59 66.04) (xy 160.02 66.04))
     (stroke (width 0) (type default))
@@
     (stroke (width 0) (type default))
   )
-  (wire (pts (xy 123.19 152.4) (xy 138.43 152.4))
+  (wire (pts (xy 123.19 152.4) (xy 130.81 152.4))
     (stroke (width 0) (type default))
   )
@@
     (stroke (width 0) (type default))
   )
+  (wire (pts (xy 130.81 152.4) (xy 138.43 152.4))
+    (stroke (width 0) (type default))
+  )
   (wire (pts (xy 90.17 60.96) (xy 100.33 60.96))
     (stroke (width 0) (type default))
   )
   (wire (pts (xy 99.06 115.57) (xy 92.71 115.57))
-    (stroke (width 0) (type default))
-  )
-  (wire (pts (xy 123.19 154.94) (xy 157.48 154.94))
     (stroke (width 0) (type default))
   )
@@
         )
       )
+    )
+  )
+  (symbol (lib_id "Device:R_US") (at 130.81 156.21 0) (unit 1)
+    (in_bom yes) (on_board yes) (dnp no) (fields_autoplaced)
+    (property "Reference" "R2" (at 133.35 154.94 0)
+      (effects (font (size 1.27 1.27)) (justify left))
+    )
+    (property "Value" "1K" (at 133.35 157.48 0)
+      (effects (font (size 1.27 1.27)) (justify left))
+    )
+    (property "Footprint" "Resistor_SMD:R_0805_2012Metric_Pad1.20x1.40mm_HandSolder" (at 131.826 156.464 90)
+      (effects (font (size 1.27 1.27)) hide)
+    )
+    (property "Datasheet" "~" (at 130.81 156.21 0)
+      (effects (font (size 1.27 1.27)) hide)
+    )
+    (pin "1")
+    (pin "2")
+    (instances
+      (project "Ackbar"
+        (path "/10d22af5-0d05-45a6-b4a8-43aad0d497f4"
+          (reference "R2") (unit 1)
+        )
+      )
